File: SlewLimiter.kicad_pcb (KiCad board)
At the start: 2 copper layers, 80 x 120 mm, 110 parts, among them J201 Conn_02x05_Odd_Even, J202 Conn_01x09, J203 Conn_01x10, J301 Conn_01x09, J302 Conn_01x10, J303 AudioJack2, J304 AudioJack2, J305 AudioJack2, J306 AudioJack2, J307 AudioJack2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

Commit message: Routed board with updated changes - pullup resistors on comparators, input to U105B goes to GND instead of -12V
Parts:
- added R125: 3.3k, Resistor_SMD:R_0402_1005Metric, F.Cu at (96.9, 109.7)
- added R126: 3.3k, Resistor_SMD:R_0402_1005Metric, F.Cu at (88.3, 117.9)
- C102, C103, C104, C105, C106, C107, C108, C109, C110, C203, C204, C205, C206: value .1u -> 100n
Connections:
- R117 pad 2: -12V -> GND
Routing:
- net -12V: track 177.7 -> 163.1 mm
- net +12V: track 184.8 -> 194.9 mm
- net Net-(R123-Pad2): track 12.4 -> 14.2 mm
- net GND: track 56.7 -> 58.3 mm, vias 22 -> 23
- net Net-(D110-Pad2): track 7.04 -> 8.47 mm
